Commit message: adding knot demo

File: sr_knot_demo/models/urdf/rope.urdf (robot description, URDF)
Before this commit: robot rope, 20 links, 19 joints
Links:
- removed link rope_seg_11
- removed link rope_seg_12
- removed link rope_seg_13
- removed link rope_seg_14
- removed link rope_seg_15
- removed link rope_seg_16
- removed link rope_seg_17
- removed link rope_seg_18
- removed link rope_seg_19
- removed link rope_seg_20
- link rope_seg_1: geometry collision cylinder length=0.051 radius=0.011; visual cylinder length=0.05 radius=0.01
- link rope_seg_10: geometry collision cylinder length=0.051 radius=0.011; visual cylinder length=0.05 radius=0.01
- link rope_seg_2: geometry collision cylinder length=0.051 radius=0.011; visual cylinder length=0.05 radius=0.01
- link rope_seg_3: geometry collision cylinder length=0.051 radius=0.011; visual cylinder length=0.05 radius=0.01
- link rope_seg_4: geometry collision cylinder length=0.051 radius=0.011; visual cylinder length=0.05 radius=0.01
- link rope_seg_5: geometry collision cylinder length=0.051 radius=0.011; visual cylinder length=0.05 radius=0.01
- link rope_seg_6: geometry collision cylinder length=0.051 radius=0.011; visual cylinder length=0.05 radius=0.01
- link rope_seg_7: geometry collision cylinder length=0.051 radius=0.011; visual cylinder length=0.05 radius=0.01
- link rope_seg_8: geometry collision cylinder length=0.051 radius=0.011; visual cylinder length=0.05 radius=0.01
- link rope_seg_9: geometry collision cylinder length=0.051 radius=0.011; visual cylinder length=0.05 radius=0.01
Joints:
- removed joint j_10
- removed joint j_11
- removed joint j_12
- removed joint j_13
- removed joint j_14
- removed joint j_15
- removed joint j_16
- removed joint j_17
- removed joint j_18
- removed joint j_19
- joint j_1: axis 1 0 0 -> 1 1 1; origin xyz=0 0 0.015 -> xyz=0 0 0.05
- joint j_2: axis 1 0 0 -> 1 1 1; origin xyz=0 0 0.015 -> xyz=0 0 0.05
- joint j_3: axis 1 0 0 -> 1 1 1; origin xyz=0 0 0.015 -> xyz=0 0 0.05
- joint j_4: axis 1 0 0 -> 1 1 1; origin xyz=0 0 0.015 -> xyz=0 0 0.05
- joint j_5: axis 1 0 0 -> 1 1 1; origin xyz=0 0 0.015 -> xyz=0 0 0.05
- joint j_6: axis 1 0 0 -> 1 1 1; origin xyz=0 0 0.015 -> xyz=0 0 0.05
- joint j_7: axis 1 0 0 -> 1 1 1; origin xyz=0 0 0.015 -> xyz=0 0 0.05
- joint j_8: axis 1 0 0 -> 1 1 1; origin xyz=0 0 0.015 -> xyz=0 0 0.05
- joint j_9: axis 1 0 0 -> 1 1 1; origin xyz=0 0 0.015 -> xyz=0 0 0.05

File: sr_knot_demo/models/xacro/link_rope.xacro (robot description, xacro)
@@ -29,4 +29,4 @@
                 </gazebo>
 </xacro:macro>
-<xacro:link_description color="Blue"/>
+<xacro:link_description color="WoodFloor"/>
 </robot>
